Commit message: 1. configured cluster 2. refined pre-sampling for b2wz1 WBC training 3. added delayed PD actuator 4. different pose command 5. z1 stl 6. high-level retrieval task for b2wz1

File: source/isaaclab_assets/data/Robots/Unitree/B2WZ1/urdf/b2wz1.urdf (robot description, URDF)
Before this commit: robot b2w_z1_description, 36 links, 35 joints
Links:
- link gripperMover: geometry collision box size=0.028 0.030 0.008; collision box size=0.028 0.030 0.008
- link gripperStator: geometry collision box size=0.028 0.030 0.008; collision box size=0.028 0.030 0.008
Joints:
- joint jointGripper: limit lower=-1.5707963267948966 upper=0.0 effort=30.0 velocity=3.1415 -> lower=-1.57079632679 upper=0.0 effort=30.0 velocity=3.1415
